File: hardware/badge/esp32-s3.kicad_sch (KiCad schematic)
At the start: 14 parts, among them SW201 TS-1187A-C-C-B, SW202 TS-1187A-C-C-B, U201 ESP32-S3-WROOM-1(N16R8)

Commit message: feat: badge v2 PCB design with panelization support
Updated schematic and PCB layout for badge v2 revision. Added
panelization project with JLCPCB production files, panelize script,
and board SVG artwork.
Changed lines of the file:
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@@
 	(text_box "UART Breakout"
 		(exclude_from_sim no)
-		(at 27.305 93.98 0)
+		(at -31.115 93.98 0)
 		(size 29.21 34.925)
 		(margins 0.9525 0.9525 0.9525 0.9525)
